File: hardware/hardware.kicad_pcb (KiCad board)
At the start: 2 copper layers, 49.7 x 46.9 mm, 5 parts, among them J1 Conn_02x03_Odd_Even, U1 CH32V003FxPx

Commit message: feat: add routes
Parts:
- added C1: 10uF, Capacitor_SMD:C_0603_1608Metric, B.Cu at (103.8, 59.6)
- added D1: LED, footprints:LYT77K-K2M1, B.Cu at (117.6, 61.0)
- added D10: LED, LED_SMD:LED_0402_1005Metric, F.Cu at (121.8, 78.1)
- added D11: LED, LED_SMD:LED_0402_1005Metric, F.Cu at (105.4, 78.1)
- added D2: LED, footprints:LYT77K-K2M1, B.Cu at (109.4, 61.0)
- added D3: LED, footprints:LYT77K-K2M1, B.Cu at (113.5, 65.1)
- added D4: LED, LED_SMD:LED_0402_1005Metric, F.Cu at (111.8, 51.6)
- added D5: LED, LED_SMD:LED_0402_1005Metric, F.Cu at (115.2, 51.6)
- added D6: LED, LED_SMD:LED_0402_1005Metric, F.Cu at (103.7, 41.7)
- added D7: LED, LED_SMD:LED_0402_1005Metric, F.Cu at (123.4, 41.7)
- added D8: LED, LED_SMD:LED_0402_1005Metric, F.Cu at (97.0, 63.7)
- added D9: LED, LED_SMD:LED_0402_1005Metric, F.Cu at (130.7, 63.7)
- added R1: 330, Resistor_SMD:R_0402_1005Metric_Pad0.72x0.64mm_HandSolder, B.Cu at (120.9, 61.5)
- added R10: 330, Resistor_SMD:R_0402_1005Metric_Pad0.72x0.64mm_HandSolder, B.Cu at (122.0, 74.7)
- added R11: 330, Resistor_SMD:R_0402_1005Metric_Pad0.72x0.64mm_HandSolder, B.Cu at (105.2, 74.7)
- added R2: 330, Resistor_SMD:R_0402_1005Metric_Pad0.72x0.64mm_HandSolder, B.Cu at (107.7, 58.5)
- added R3: 330, Resistor_SMD:R_0402_1005Metric_Pad0.72x0.64mm_HandSolder, B.Cu at (113.6, 67.3)
- added R4: 330, Resistor_SMD:R_0402_1005Metric_Pad0.72x0.64mm_HandSolder, B.Cu at (108.6, 52.1)
- added R5: 330, Resistor_SMD:R_0402_1005Metric_Pad0.72x0.64mm_HandSolder, B.Cu at (108.6, 53.0)
- added R6: 330, Resistor_SMD:R_0402_1005Metric_Pad0.72x0.64mm_HandSolder, B.Cu at (101.0, 43.4)
- added R7: 330, Resistor_SMD:R_0402_1005Metric_Pad0.72x0.64mm_HandSolder, B.Cu at (125.9, 43.4)
- added R8: 330, Resistor_SMD:R_0402_1005Metric_Pad0.72x0.64mm_HandSolder, B.Cu at (100.0, 63.7)
- added R9: 330, Resistor_SMD:R_0402_1005Metric_Pad0.72x0.64mm_HandSolder, B.Cu at (127.8, 63.7)
Connections:
- U1 pad 1: unconnected-(U1-PD4-Pad1) -> /LED_4
- U1 pad 10: unconnected-(U1-PC0-Pad10) -> /LED_7
- U1 pad 11: unconnected-(U1-PC1-Pad11) -> /LED_5
- U1 pad 12: unconnected-(U1-PC2-Pad12) -> /LED_8
- U1 pad 2: unconnected-(U1-PD5-Pad2) -> /LED_1
- U1 pad 20: unconnected-(U1-PD3-Pad20) -> /LED_3
- U1 pad 3: unconnected-(U1-PD6-Pad3) -> /LED_2
- U1 pad 4: unconnected-(U1-PD7-Pad4) -> /LED_6
- U1 pad 5: unconnected-(U1-PA1-Pad5) -> /RIGHT_EYE
- U1 pad 6: unconnected-(U1-PA2-Pad6) -> /NOSE
- U1 pad 8: unconnected-(U1-PD0-Pad8) -> /LEFT_EYE
Routing:
- net /SWDIO: track 0.00 -> 41.2 mm
- net /LED_7: track 0.00 -> 32.0 mm
- net /LED_6: track 0.00 -> 31.5 mm
- net /LED_4: track 0.00 -> 28.9 mm
- net +3.3V: track 0.00 -> 25.3 mm, vias 0 -> 2
- net /LED_8: track 0.00 -> 21.7 mm
- net /NOSE: track 0.00 -> 17.4 mm
- net /RIGHT_EYE: track 0.00 -> 15.6 mm
- net /LED_3: track 0.00 -> 9.06 mm
- net /LED_5: track 0.00 -> 7.04 mm
- net Net-(D5-A): track 0.00 -> 6.77 mm, vias 0 -> 1
- net /LEFT_EYE: track 0.00 -> 4.25 mm
- net /LED_1: track 0.00 -> 3.66 mm
- net Net-(D3-K): track 0.00 -> 3.57 mm
- net /LED_2: track 0.00 -> 3.53 mm
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
Commit message: feat: add vias
Routing:
- net GND: vias 22 -> 23
Changed lines of the file:
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@@
 			(at 0 4.2 0)
 			(layer "B.SilkS")
+			(hide yes)
 			(effects
 				(font
@@
 			(at 0 1.43 0)
 			(layer "B.SilkS")
+			(hide yes)
 			(effects
 				(font
@@
 	)
 	(via
-		(at 102.91 53.6)
+		(at 120.1 50.5)
 		(size 0.6)
 		(drill 0.3)
@@
 	)
 	(via
+		(at 106.64 50.43)
+		(size 0.6)
+		(drill 0.3)
+		(layers "F.Cu" "B.Cu")
+		(free yes)
+		(net 5)
+	)
+	(via
 		(at 97 66.5)
 		(size 0.6)
@@
 	)
 	(via
-		(at 113.55 60.98)
+		(at 114.52 60.96)
 		(size 0.6)
 		(drill 0.3)
